Commit message: 整合代码，给他加了tf2

File: src/rm_gimbal_description/urdf/rm_gimbal.urdf.xacro (robot description, xacro)
@@ -5,4 +5,6 @@
   <xacro:arg name="xyz_muzzle" default="0 0 0.45" />
   <xacro:arg name="rpy" default="0 0 0" />
+  <xacro:arg name="xyz_lidar" default="0 0 0.18" />
+  <xacro:arg name="rpy_lidar" default="0 0 0" />
   <link name="chassis_link" />
   <link name="muzzle_link" />
@@ -15,5 +17,5 @@
   <joint name="camera_joint" type="fixed">
     <origin xyz="$(arg xyz_camera)" rpy="$(arg rpy)" />
-    <parent link="chassis_link" />
+    <parent link="muzzle_link" />
     <child link="camera_link" />
     <axis xyz="0 0 0" />
@@ -25,3 +27,9 @@
     <child link="camera_optical_frame" />
   </joint>
+  <link name="livox_frame" />
+  <joint name="lidar_joint" type="fixed">
+    <origin xyz="$(arg xyz_lidar)" rpy="$(arg rpy_lidar)" />
+    <parent link="muzzle_link" />
+    <child link="livox_frame" />
+  </joint>
 </robot>

Commit message: 完善雷达的检测机制

File: src/rm_gimbal_description/urdf/rm_gimbal.urdf.xacro (robot description, xacro)
@@ -30,5 +30,5 @@
   <joint name="lidar_joint" type="fixed">
     <origin xyz="$(arg xyz_lidar)" rpy="$(arg rpy_lidar)" />
-    <parent link="muzzle_link" />
+    <parent link="camera_optical_joint" />
     <child link="livox_frame" />
   </joint>
